File: ButtonBreakout.sch (EAGLE design)
At the start: 56 parts, among them IC1 74HC595D, Q1 FDN360P, Q4 FDN360P, Q5 FDN360P, X1 JST-XH-02-PIN-LONG-PAD, X10 JST-XH-04-PIN-LONG-PAD, X11 JST-XH-04-PIN-LONG-PAD, X12 JST-XH-04-PIN-LONG-PAD, X13 JST-XH-04-PIN-LONG-PAD, X14 JST-XH-06-PIN-LONG-PAD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

Commit message: USBPD design review
Parts:
- D1, D2, D3, D4, D5, D6, D7, D8, D9: value (none) -> SS34; device adafruit:DIODESOD-123 -> tmc:SS34
- H1, H2: value MOUNT-HOLE3.6 -> MOUNT-HOLE3.0; device holes:MOUNT-HOLE3.6 -> holes:MOUNT-HOLE3.0
- Q1, Q4, Q5: value FDN360P -> AO3414SOT23; device transistor-power:FDN360P -> tmc:AO3414SOT23
- Q2, Q3, Q6: value (none) -> AO3414SOT23; device adafruit:MOSFET-NREFLOW -> tmc:AO3414SOT23
- Q7, Q8, Q9: value (none) -> AO3415; device adafruit:MOSFET-NREFLOW -> tmc:AO3415
Connections:
- net +12V: now also Q7.S, Q8.S, Q9.S; no longer Q1.S, Q4.S, Q5.S
- net ANODE0: now also Q7.D; no longer Q4.D
- net ANODE1: now also Q8.D; no longer Q1.D
- net ANODE2: now also Q9.D; no longer Q5.D
- net CATHODE0: now also Q1.D; no longer Q3.D
- net CATHODE1: now also Q2.D; no longer Q8.D
- net CATHODE2: now also Q3.D; no longer Q9.D
- net GND: now also Q1.S, Q4.S, Q5.S; no longer Q7.S, Q8.S, Q9.S
- net N$1: now also Q2.G; no longer Q8.G
- net N$16: now also Q4.G; no longer Q6.G
- net N$17: now also Q6.D, Q9.G; no longer Q5.G, Q7.D
- net N$18: now also Q6.G; no longer Q7.G
- net N$2: now also Q3.G; no longer Q9.G
- net N$3: now also Q5.D, Q8.G; no longer Q1.G, Q2.D
- net N$4: now also Q5.G; no longer Q2.G
- net N$5: now also Q1.G; no longer Q3.G
- net N$6: now also Q4.D, Q7.G; no longer Q4.G, Q6.D
Other:
- moved on the sheet: Q2, Q3, Q6
