File: ButtonBreakout.brd (EAGLE design)
At the start: 62.9 x 76.2 mm, 56 parts, among them IC1 74HC595D, Q1 FDN360P, Q4 FDN360P, Q5 FDN360P, X1 JST-XH-02-PIN-LONG-PAD, X10 JST-XH-04-PIN-LONG-PAD, X11 JST-XH-04-PIN-LONG-PAD, X12 JST-XH-04-PIN-LONG-PAD, X13 JST-XH-04-PIN-LONG-PAD, X14 JST-XH-06-PIN-LONG-PAD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

Commit message: USBPD design review
Parts:
- D1, D2, D3, D4, D5, D6, D7, D8, D9: value (none) -> SS34; device adafruit:SOD-123 -> tmc:SMA
- H1, H2: value MOUNT-HOLE3.6 -> MOUNT-HOLE3.0; device holes:3,6 -> holes:3,0
- Q1, Q4, Q5: value FDN360P -> AO3414SOT23; device transistor-power:SUPER-SOT3 -> tmc:SOT95P240X110-3N
- Q2, Q3, Q6: value (none) -> AO3414SOT23; device adafruit:SOT23 -> tmc:SOT95P240X110-3N
- Q7, Q8, Q9: value (none) -> AO3415; device adafruit:SOT23 -> tmc:SOT95P240X110-3N
- moved Q9 59.0 mm to (45.1, 58.4), turned to 270 degrees
- moved Q2 42.7 mm to (6.99, 26.7), turned to 270 degrees
- moved Q8 40.7 mm to (32.4, 58.4), turned to 270 degrees
- moved Q3 34.3 mm to (6.99, 13.3), turned to 270 degrees
- moved Q7 28.6 mm to (19.7, 58.4), turned to 270 degrees
- moved Q1 27.0 mm to (6.99, 47.6), turned to 270 degrees
- moved Q6 26.0 mm to (48.9, 58.4), turned to 270 degrees
- moved Q5 8.26 mm to (36.2, 58.4), turned to 270 degrees
- moved Q4 4.45 mm to (23.5, 58.4), turned to 270 degrees
- moved X14 2.54 mm to (57.1, 11.4)
- moved D6 1.80 mm to (47.0, 25.4)
- moved D1 1.80 mm to (21.6, 46.4)
- moved D4 1.80 mm to (21.6, 25.4)
- moved D2 1.80 mm to (34.3, 46.4)
- moved D7 1.80 mm to (21.6, 4.45)
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Connections:
- net +12V: now also Q7.2, Q8.2, Q9.2; no longer Q1.2, Q4.2, Q5.2
- net ANODE0: now also Q7.3; no longer Q4.3
- net ANODE1: now also Q8.3; no longer Q1.3
- net ANODE2: now also Q9.3; no longer Q5.3
- net CATHODE0: now also Q1.3; no longer Q3.3
- net CATHODE1: now also Q2.3; no longer Q8.3
- net CATHODE2: now also Q3.3; no longer Q9.3
- net GND: now also Q1.2, Q4.2, Q5.2; no longer Q7.2, Q8.2, Q9.2
- net N$1: now also Q2.1; no longer Q8.1
- net N$16: now also Q4.1; no longer Q6.1
- net N$17: now also Q6.3, Q9.1; no longer Q5.1, Q7.3
- net N$18: now also Q6.1; no longer Q7.1
- net N$2: now also Q3.1; no longer Q9.1
- net N$3: now also Q5.3, Q8.1; no longer Q1.1, Q2.3
- net N$4: now also Q5.1; no longer Q2.1
- net N$5: now also Q1.1; no longer Q3.1
- net N$6: now also Q4.3, Q7.1; no longer Q4.1, Q6.3
Routing:
- net B_COL2: track 59.4 -> 75.6 mm, vias 1 -> 0
- net B_ROW2: track 59.4 -> 66.4 mm
- net B_ROW0: track 80.9 -> 87.5 mm
- net B_COL0: track 89.4 -> 84.0 mm
- net GND: track 28.2 -> 25.1 mm, vias 17 -> 14
- net ANODE2: track 64.1 -> 66.8 mm
- net ANODE1: track 59.2 -> 61.7 mm
- net N$12: track 5.96 -> 7.21 mm
- net N$7: track 5.96 -> 7.21 mm
- net N$8: track 5.96 -> 7.21 mm
- net N$11: track 5.96 -> 7.21 mm
- net N$10: track 5.96 -> 7.21 mm
- net N$13: track 5.96 -> 7.21 mm
- net N$14: track 5.96 -> 7.21 mm
- net +12V: track 67.3 -> 66.3 mm
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
Commit message: Board Redone with notes from Ben
Routing:
- net B_ROW2: track 66.4 -> 42.8 mm
- net B_COL2: track 75.6 -> 55.4 mm, vias 0 -> 4
- net B_ROW0: track 87.5 -> 72.4 mm, vias 1 -> 2
- net B_ROW1: track 64.3 -> 52.9 mm, vias 1 -> 0
- net LCOL2: track 54.5 -> 43.6 mm
- net B_COL0: track 84.0 -> 91.2 mm, vias 4 -> 6
- net LCOL0: track 19.3 -> 25.8 mm, vias 0 -> 2
- net ANODE2: track 66.8 -> 61.5 mm, vias 2 -> 4
- net LATCH: track 45.8 -> 42.7 mm, vias 0 -> 2
- net B_COL1: track 74.3 -> 71.6 mm
- net ANODE0: track 59.9 -> 62.5 mm
- net OEN: track 51.0 -> 48.9 mm, vias 0 -> 2
- net +5V: track 41.4 -> 43.6 mm
- net CATHODE2: track 36.4 -> 38.2 mm
- net LCOL1: track 37.3 -> 35.8 mm, vias 0 -> 2
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Other:
- board text added: "Tim Chase Julia Sorrentino Brad Piva Josh Steakelum Fall 2019 Speed Of Light Controller github.com/timChase98/SpeedOfLightContoller"
