File: SpeedOfLightController.sch (EAGLE design)
At the start: 140 parts, among them IC10 74LS595D, IC11 74LS595D, Q10 FDN360P, Q12 FDN360P, Q14 FDN360P, Q16 FDN360P, Q18 FDN360P, Q20 FDN360P, Q22 FDN360P, Q24 FDN360P, Q26 FDN360P, SW2 MOMENTARYBUTTON, U1 ATMEGA328PBTQFP-32, U2 LM380NDIP14, U3 AD5111ADLFCSP10, X1 JST-XH-08-PIN-LONG-PAD, X10 JST-XH-06-PIN-LONG-PAD, X11 JST-XH-06-PIN-LONG-PAD, X12 JST-XH-06-PIN-LONG-PAD, X13 JST-XH-06-PIN-LONG-PAD, X14 JST-XH-07-PIN-LONG-PAD, X15 JST-XH-02-PIN-LONG-PAD, X16 JST-XH-02-PIN-LONG-PAD, X17 JST-XH-02-PIN-LONG-PAD, X18 JST-XH-02-PIN-LONG-PAD, X19 JST-XH-03-PIN-LONG-PAD, X2 JST-XH-08-PIN-LONG-PAD, X20 JST-XH-03-PIN-LONG-PAD, X21 JST-XH-03-PIN-LONG-PAD, X22 JST-XH-03-PIN-LONG-PAD, X3 JST-XH-08-PIN-LONG-PAD, X4 JST-XH-08-PIN-LONG-PAD, X5 JST-XH-08-PIN-LONG-PAD, X6 JST-XH-08-PIN-LONG-PAD, X7 JST-XH-08-PIN-LONG-PAD, X8 JST-XH-08-PIN-LONG-PAD, X9 JST-XH-08-PIN-LONG-PAD

Commit message: USBPD design review
Parts:
- removed CN1: (no value), adafruit:USBMINIB
- removed F3: FIDUCIAL, ECE388:FIDUCIAL
- removed JP13: (no value), pinhead:PINHD-1X5
- removed JP14: (no value), pinhead:PINHD-1X3
- removed R5: 82K, rcl:R-EU_R0805
- removed X27: (no value), ECE388:1X02_5MM_SCREW
- added C14, C15: 0.1uF, rcl:C-EUC0805
- added C16: 680uF, rcl:CPOL-US140CLH-0810
- added C17: 220uF, rcl:CPOL-US140CLH-0810
- added H1, H2: MOUNT-HOLE3.0, holes:MOUNT-HOLE3.0
- added IC3: (no value), linear:LM2596S
- added J1: 6_PIN_SERIAL_CABLEPTH, SparkFun-Connectors:6_PIN_SERIAL_CABLEPTH
- added JP10: (no value), pinhead:PINHD-1X3
- added JP2: JUMPER-SMT_3_1-NC_TRACE_SILK, SparkFun-Jumpers:JUMPER-SMT_3_1-NC_TRACE_SILK
- added JP5: (no value), pinhead:PINHD-1X5
- added JP6: (no value), pinhead:PINHD-1X4
- added JP7, JP8, JP9: (no value), pinhead:PINHD-1X1
- added R59, R62: 1K5, rcl:R-EU_R0805
- added R60, R63: 470, rcl:R-EU_R0805
- added R61: 10K, rcl:R-EU_R0805
- added SJ1, SJ3: (no value), ECE388:SJ
- added SJ4, SJ5: (no value), jumper:SJ2WW
- added U4: AD5141ADLFCSP3, tmc:AD5141ADLFCSP3
- added X25: JST-XH-03-PIN-LONG-PAD, Rembrandt Electronics - JST XH Connectors v1-0:JST-XH-03-PIN-LONG-PAD
- C1, C4: value (none) -> 0.1uF
- C10, C12: value (none) -> 470uF; device rcl:C-EUC0805 -> rcl:CPOL-US140CLH-0810
- C11: value (none) -> 47uF
- C13: value (none) -> 4.7uF
- C2, C3: value (none) -> 22pF
- C7: value 22uF -> 0.1uF
- C8: value 22uF -> 47nF
- C9: value (none) -> 47nF
- F1: value (none) -> FIDUCIAL; device adafruit:PTCFUSE-1812 -> ECE388:FIDUCIAL
- JP1: value (none) -> JUMPER-SMT_3_1-NC_TRACE_SILK; device pinhead:PINHD-2X3 -> SparkFun-Jumpers:JUMPER-SMT_3_1-NC_TRACE_SILK
- Q1: value (none) -> 16MHz
- Q10, Q14, Q16, Q20, Q22, Q24, Q26: value FDN360P -> AO3414SOT23; device transistor-power:FDN360P -> tmc:AO3414SOT23
- Q11, Q13, Q17, Q19, Q5, Q6, Q7: value (none) -> AO3415; device adafruit:MOSFET-NREFLOW -> tmc:AO3415
- Q12, Q18: value FDN360P -> AO3415; device transistor-power:FDN360P -> tmc:AO3415
- Q15, Q2, Q21, Q23, Q25, Q3, Q4, Q8, Q9: value (none) -> AO3414SOT23; device adafruit:MOSFET-NREFLOW -> tmc:AO3414SOT23
- R11, R17, R23, R29, R35, R41, R49, R51, R55: value 1K -> 10K
- R14, R20, R26, R32, R38, R44, R46, R54, R8: value 10K -> 1K
- R57: value 10K -> 0; device rcl:R-EU_R0805 -> rcl:R-EU_R0805W
- R6: value 4.3K -> 10K
- SJ2: device jumper:SJ2W -> jumper:SJ2WW
- U$1: value MT3608SOT23-6 -> USBMICRO; device tmc:MT3608SOT23-6 -> tmc:USBMICRO
- U3: value AD5111ADLFCSP10 -> SSM2305ADMSOP8_2; device tmc:AD5111ADLFCSP10 -> tmc:SSM2305ADMSOP8_2
- X1, X2, X4, X5: value JST-XH-08-PIN-LONG-PAD -> JST-XH-06-PIN-LONG-PAD; device Rembrandt Electronics - JST XH Connectors v1-0:JST-XH-08-PIN-LONG-PAD -> Rembrandt Electronics - JST XH Connectors v1-0:JST-XH-06-PIN-LONG-PAD
- X10, X11, X12, X13: value JST-XH-06-PIN-LONG-PAD -> JST-XH-08-PIN-LONG-PAD; device Rembrandt Electronics - JST XH Connectors v1-0:JST-XH-06-PIN-LONG-PAD -> Rembrandt Electronics - JST XH Connectors v1-0:JST-XH-08-PIN-LONG-PAD
- X14: value JST-XH-07-PIN-LONG-PAD -> JST-XH-08-PIN-LONG-PAD; device Rembrandt Electronics - JST XH Connectors v1-0:JST-XH-07-PIN-LONG-PAD -> Rembrandt Electronics - JST XH Connectors v1-0:JST-XH-08-PIN-LONG-PAD
- X15, X16, X17: value JST-XH-02-PIN-LONG-PAD -> (none); device Rembrandt Electronics - JST XH Connectors v1-0:JST-XH-02-PIN-LONG-PAD -> ECE388:1X02_5MM_SCREW
- X19, X20, X21: value JST-XH-03-PIN-LONG-PAD -> JST-XH-02-PIN-LONG-PAD; device Rembrandt Electronics - JST XH Connectors v1-0:JST-XH-03-PIN-LONG-PAD -> Rembrandt Electronics - JST XH Connectors v1-0:JST-XH-02-PIN-LONG-PAD
- X23, X24: value (none) -> JST-XH-03-PIN-LONG-PAD; device ECE388:1X02_5MM_SCREW -> Rembrandt Electronics - JST XH Connectors v1-0:JST-XH-03-PIN-LONG-PAD
- X3: value JST-XH-08-PIN-LONG-PAD -> JST-XH-07-PIN-LONG-PAD; device Rembrandt Electronics - JST XH Connectors v1-0:JST-XH-08-PIN-LONG-PAD -> Rembrandt Electronics - JST XH Connectors v1-0:JST-XH-07-PIN-LONG-PAD
- renumbered IC10 to IC1, IC11 to IC2, SW2 to SW1
Connections:
- removed net N$26: C11.2, X23-1.KL
- removed net N$33: C7.1, D1.C, F1.1, R5.2
- removed net SOUND_C: R58.1, U1.PE0, U3.CLK
- removed net SOUND_UD: U1.PE3, U3.UD
- new net ADSOUND+: SJ4.1, U3.OUT+
- new net ADSOUND-: SJ5.3, U3.OUT-
- new net D+: JP5.3, R58.1, R59.2, R60.2, U$1.D+
- new net D-: JP5.2, R61.2, R62.1, R63.1, U$1.D-
- new net FTDIRX: J1.3, JP1.2
- new net FTDITX: J1.2, JP2.2
- new net LMSOUND: C12.-, SJ4.3
- new net N$40: IC3.EN, SJ2.2
- new net N$41: C17.+, IC3.FB, L1.2, SJ3.2
- new net SOUND+: SJ4.2, X15-1.KL
- new net SOUND-: SJ5.2, X16-2.KL
- new net UCD+: R60.1, U1.PE1
- new net UCD-: R63.2, U1.PE0
- net +12V: now also C16.+, IC3.IN, JP10.2, Q11.S, Q13.S, Q17.S, Q19.S, Q5.S, Q6.S, Q7.S, R13.2, R14.2, R15.2, R25.2, R26.2, R37.2, R38.2, SJ1.2, SJ2.3, X17-1.KL, X19-1.S, X19-2.S, X20-1.S, X20-2.S, X21-1.S, X21-2.S; no longer F1.2, JP14.2, Q10.S, Q14.S, Q16.S, Q20.S, Q22.S, Q24.S, Q26.S, R23.2, R31.2, R35.2, R43.2, R47.2, R51.2, R55.2, X15-1.S, X15-2.S, X16-1.S, X16-2.S, X17-1.S, X17-2.S, X27-1.KL
- net +5V: now also C10.+, C14.2, C15.1, C4.2, C6.1, C7.1, J1.4, JP10.1, R4.2, R6.2, R61.1, SJ3.1, U3.SHDWN, U3.VDD, U4.LRDAC, U4.VDD, U4.VLOGIC, U4.WP, X3-1.S; no longer C1.1, C12.2, C2.1, C8.1, C9.1, CN1.VBUS, JP1.5, JP13.1, JP14.1, L1.1, R3.2, R57.2, SJ2.3, U$1.VIN, U3.VCC, X14-1.S
- net A: now also Q20.D, X10-5.S, X11-5.S, X12-5.S, X13-5.S, X14-5.S; no longer Q4.D, X1-5.S, X2-5.S, X3-5.S, X4-5.S, X5-5.S
- net AN1: now also R7.1; no longer R21.1
- net AN2: now also R19.1; no longer R25.1
- net AN3: now also R31.1; no longer R29.1
- net AN4: now also R8.1; no longer R33.1
- net AN5: now also R20.1; no longer R37.1
- net AN6: now also R32.1; no longer R41.1
- net AN7: now also R9.1; no longer R45.1
- net AN8: now also R21.1; no longer R49.1
- net AN9: now also R33.1; no longer R53.1
- net B: now also Q21.D, X10-6.S, X11-6.S, X12-6.S, X13-6.S, X14-6.S; no longer Q2.D, X1-6.S, X2-6.S, X3-6.S, X4-6.S, X5-6.S
- net B_COL_0: now also X1-4.S, X2-4.S; no longer X10-4.S, X11-4.S
- net B_COL_1: now also X1-5.S, X2-5.S; no longer X10-5.S, X11-5.S
- net B_COL_2: now also X1-6.S, X2-6.S; no longer X10-6.S, X11-6.S
- net B_COL_3: now also X4-4.S, X5-4.S; no longer X12-4.S, X13-4.S
- net B_COL_4: now also X4-5.S, X5-5.S; no longer X12-5.S, X13-5.S
- net B_COL_5: now also X4-6.S, X5-6.S; no longer X12-6.S, X13-6.S
- net B_ROW_0: now also X1-1.S, X4-1.S; no longer X10-1.S, X12-1.S
- net B_ROW_1: now also X1-2.S, X4-2.S; no longer X10-2.S, X12-2.S
- net B_ROW_2: now also X1-3.S, X4-3.S; no longer X10-3.S, X12-3.S
- net B_ROW_3: now also X2-1.S, X5-1.S; no longer X11-1.S, X13-1.S
- net B_ROW_4: now also X2-2.S, X5-2.S; no longer X11-2.S, X13-2.S
- net B_ROW_5: now also X2-3.S, X5-3.S; no longer X11-3.S, X13-3.S
- net C: now also Q22.D, X10-7.S, X11-7.S, X12-7.S, X13-7.S, X14-7.S; no longer Q3.D, X1-7.S, X2-7.S, X3-7.S, X4-7.S, X5-7.S
- net D: now also Q23.D, X10-1.S, X11-1.S, X12-1.S, X13-1.S, X14-1.S; no longer Q5.D, X1-1.S, X2-1.S, X3-1.S, X4-1.S, X5-1.S
- net DTR: now also C1.2, J1.1; no longer C6.2, JP1.6
- net E: now also Q24.D, X10-2.S, X11-2.S, X12-2.S, X13-2.S, X14-2.S; no longer Q6.D, X1-2.S, X2-2.S, X3-2.S, X4-2.S, X5-2.S
- net F: now also Q25.D, X10-4.S, X11-4.S, X12-4.S, X13-4.S, X14-4.S; no longer Q7.D, X1-4.S, X2-4.S, X3-4.S, X4-4.S, X5-4.S
- net G: now also Q26.D, X10-3.S, X11-3.S, X12-3.S, X13-3.S, X14-3.S; no longer Q8.D, X1-3.S, X2-3.S, X3-3.S, X4-3.S, X5-3.S
- net GND: now also C10.-, C11.2, C14.1, C15.2, C16.-, C17.-, C2.1, C6.2, C9.1, D1.A, IC3.GND, IC3.GND@1, J1.5, J1.6, JP10.3, JP5.5, JP6.1, JP6.2, JP6.3, JP6.4, JP7.1, JP8.1, JP9.1, Q10.S, Q14.S, Q16.S, Q20.S, Q22.S, Q24.S, Q26.S, R11.1, R17.1, R23.1, R29.1, R3.1, R35.1, R41.1, R49.1, R51.1, R55.1, R57.1, R59.1, R62.2, SJ5.1, U4.DIS, U4.GND, U4.INDEP, U4.RESET, U4.VSS, X17-2.KL, X23-1.S, X23-2.S, X23-3.S, X24-1.S, X24-2.S, X24-3.S, X25-1.S, X25-2.S, X25-3.S, X3-7.S; no longer C1.2, C10.2, C12.1, C2.2, C8.2, C9.2, CN1.GND, JP1.1, JP1.3, JP13.5, JP14.3, Q11.S, Q13.S, Q17.S, Q19.S, Q5.S, Q6.S, Q7.S, R14.1, R20.1, R26.1, R32.1, R38.1, R4.1, R44.1, R46.1, R54.1, R6.1, R8.1, U3.B, X14-7.S, X19-1.S, X19-2.S, X19-3.S, X20-1.S, X20-2.S, X20-3.S, X21-1.S, X21-2.S, X21-3.S, X24-2.KL, X27-2.KL
- net LED_B: now also X3-5.S; no longer X14-5.S
- net LED_D_OUT: now also X3-2.S; no longer X14-2.S
- net LED_L: now also X3-4.S; no longer X14-4.S
- net LED_O: now also R3.2, X3-6.S; no longer R4.2, X14-6.S
- net MISO: now also U4.SDO_AD1
- net MOSI: now also U4.SDI_SDA
- net N$1: now also Q21.G, R44.2, R49.2; no longer Q2.G, R7.2, R8.2
- net N$10: now also Q14.G, R31.2, R34.2; no longer Q13.G, R29.2, R30.2
- net N$11: now also Q3.G, R11.2, R8.2; no longer Q15.G, R33.2, R34.2
- net N$12: now also Q9.G, R20.2, R23.2; no longer Q17.G, R37.2, R38.2
- net N$13: now also Q15.G, R32.2, R35.2; no longer Q19.G, R41.2, R42.2
- net N$14: now also Q4.G, R12.2, R9.2; no longer Q21.G, R45.2, R46.2
- net N$15: now also Q10.G, R21.2, R24.2; no longer Q23.G, R49.2, R50.2
- net N$16: now also Q16.G, R33.2, R36.2; no longer Q25.G, R53.2, R54.2
- net N$17: now also C2.2; no longer C3.2
- net N$18: now also C3.2; no longer C4.2
- net N$19: now also JP5.1, SJ1.1, U$1.+5; no longer R5.1, R6.2, U$1.FB
- net N$2: now also Q22.G, R45.2, R50.2; no longer Q3.G, R10.2, R9.2
- net N$20: now also X15-2.KL, X16-1.KL; no longer X23-2.KL, X24-1.KL
- net N$21: now also C12.+, U2.OUT; no longer CN1.D+, JP13.2
- net N$22: now also C11.1; no longer C10.1
- net N$23: now also C9.2, U3.IN-; no longer CN1.D-, JP13.3
- net N$24: now also C8.2, U3.IN+; no longer D1.A, L1.2, U$1.SW
- net N$25: now also R57.2, U4.B; no longer C11.1, U2.OUT
- net N$27: now also Q16.D, Q19.G, R39.1; no longer Q25.D, Q26.G, R55.1
- net N$28: now also Q10.D, Q13.G, R27.1; no longer Q23.D, Q24.G, R51.1
- net N$29: now also Q4.D, Q7.G, R15.1; no longer Q21.D, Q22.G, R47.1
- net N$3: now also Q23.G, R46.2, R51.2; no longer Q5.G, R11.2, R12.2
- net N$30: now also Q3.D, Q6.G, R14.1; no longer Q15.D, Q16.G, R35.1
- net N$31: now also JP5.4, U$1.ID; no longer CN1.ID, JP13.4
- net N$32: now also D1.C, IC3.OUT, L1.1; no longer SJ2.2, U$1.EN
- net N$34: now also Q12.G, Q9.D, R26.1; no longer Q17.D, Q18.G, R39.1
- net N$35: now also Q15.D, Q18.G, R38.1; no longer Q19.D, Q20.G, R43.1
- net N$36: now also Q14.D, Q17.G, R37.1; no longer Q13.D, Q14.G, R31.1
- net N$37: now also Q11.G, Q8.D, R25.1; no longer Q11.D, Q12.G, R27.1
- net N$38: now also Q2.D, Q5.G, R13.1; no longer Q10.G, Q9.D, R23.1
- net N$4: now also Q24.G, R47.2, R52.2; no longer Q6.G, R15.2, R16.2
- net N$5: now also Q20.G, R43.2, R48.2; no longer Q4.G, R13.2, R14.2
- net N$6: now also Q25.G, R53.2, R55.2; no longer Q7.G, R17.2, R18.2
- net N$7: now also Q26.G, R54.2, R56.2; no longer Q8.G, R19.2, R20.2
- net N$8: now also Q2.G, R10.2, R7.2; no longer Q9.G, R21.2, R22.2
- net N$9: now also Q8.G, R19.2, R22.2; no longer Q11.G, R25.2, R26.2
- net RX: now also JP1.3, JP2.1; no longer JP1.2
- net SCK: now also U4.SCLK_SCL, X3-3.S; no longer X14-3.S
- net SCORE0_1: now also Q5.D, R16.2, X6-8.S; no longer Q10.D, R24.2, X1-8.S
- net SCORE0_10: now also Q11.D, X7-8.S; no longer Q12.D, X2-8.S
- net SCORE0_100: now also Q17.D, R40.2, X8-8.S; no longer Q14.D, R32.2, X3-8.S
- net SCORE1_1: now also Q6.D, R17.2, X9-8.S; no longer Q16.D, R36.2, X4-8.S
- net SCORE1_10: now also Q12.D, R29.2, X10-8.S; no longer Q18.D, R40.2, X5-8.S
- net SCORE1_100: now also Q18.D, R41.2, X11-8.S; no longer Q20.D, R44.2, X6-8.S
- net SCORE2_1: now also Q7.D, R18.2, X12-8.S; no longer Q22.D, R48.2, X7-8.S
- net SCORE2_10: now also Q13.D, R30.2, X13-8.S; no longer Q24.D, R52.2, X8-8.S
- net SCORE2_100: now also Q19.D, R42.2, X14-8.S; no longer Q26.D, R56.2, X9-8.S
- net SIGA: now also R43.1; no longer R13.1
- net SIGB: now also R44.1; no longer R7.1
- net SIGC: now also R45.1; no longer R9.1
- net SIGD: now also R46.1; no longer R11.1
- net SIGE: now also R47.1; no longer R15.1
- net SIGF: now also R53.1; no longer R17.1
- net SIGG: now also R54.1; no longer R19.1
- net SOUNDOUT: now also U4.A; no longer U3.A
- net SOUND_ATND: now also C8.1, U4.W; no longer U3.W
- net SOUND_CS: now also R4.1, U1.PE3, U4.SY_AD0; no longer R57.1, U1.PE1, U3.CS
- net TX: now also JP1.1, JP2.3; no longer JP1.4
- net UC_RESET: now also C1.1, R6.1; no longer C6.1, R3.1
Other:
- note added: "LM2569"
- note added: "USB QC set resistors"
- note removed: "GND CTS VCC"
- note removed: "TXO RXI DTR"

Commit message: Change to 100mm square board
Parts:
- removed JP7, JP8, JP9: (no value), pinhead:PINHD-1X1
- removed X17: (no value), ECE388:1X02_5MM_SCREW
- added SJ6: (no value), ECE388:SJ
Connections:
- net +12V: no longer X17-1.KL
- net GND: no longer JP7.1, JP8.1, JP9.1, X17-2.KL
- net SOUNDOUT: now also SJ6.2
- net SOUND_ATND: now also SJ6.1
- net UCD+: now also U1.PE0; no longer U1.PE1
- net UCD-: now also U1.PE1; no longer U1.PE0
Changed lines of the file:
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@@
 <part name="P+37" library="supply1" library_urn="urn:adsk.eagle:library:371" deviceset="+12V" device=""/>
 <part name="SJ1" library="ECE388" deviceset="SJ" device=""/>
-<part name="X17" library="ECE388" deviceset="1X02_5MM_SCREW" device=""/>
-<part name="P+41" library="supply1" library_urn="urn:adsk.eagle:library:371" deviceset="+12V" device=""/>
-<part name="SUPPLY73" library="supply2" library_urn="urn:adsk.eagle:library:372" deviceset="GND" device=""/>
 <part name="R58" library="rcl" library_urn="urn:adsk.eagle:library:334" deviceset="R-EU_" device="R0805" package3d_urn="urn:adsk.eagle:package:23553/2" value="10K"/>
 <part name="R59" library="rcl" library_urn="urn:adsk.eagle:library:334" deviceset="R-EU_" device="R0805" package3d_urn="urn:adsk.eagle:package:23553/2" value="1K5"/>
@@
 <part name="JP6" library="pinhead" library_urn="urn:adsk.eagle:library:325" deviceset="PINHD-1X4" device="" package3d_urn="urn:adsk.eagle:package:22407/2"/>
 <part name="SUPPLY75" library="supply2" library_urn="urn:adsk.eagle:library:372" deviceset="GND" device=""/>
-<part name="JP9" library="pinhead" library_urn="urn:adsk.eagle:library:325" deviceset="PINHD-1X1" device="" package3d_urn="urn:adsk.eagle:package:22485/2"/>
-<part name="SUPPLY78" library="supply2" library_urn="urn:adsk.eagle:library:372" deviceset="GND" device=""/>
-<part name="JP8" library="pinhead" library_urn="urn:adsk.eagle:library:325" deviceset="PINHD-1X1" device="" package3d_urn="urn:adsk.eagle:package:22485/2"/>
-<part name="SUPPLY77" library="supply2" library_urn="urn:adsk.eagle:library:372" deviceset="GND" device=""/>
-<part name="JP7" library="pinhead" library_urn="urn:adsk.eagle:library:325" deviceset="PINHD-1X1" device="" package3d_urn="urn:adsk.eagle:package:22485/2"/>
-<part name="SUPPLY76" library="supply2" library_urn="urn:adsk.eagle:library:372" deviceset="GND" device=""/>
 <part name="J1" library="SparkFun-Connectors" library_urn="urn:adsk.eagle:library:513" deviceset="6_PIN_SERIAL_CABLE" device="PTH" package3d_urn="urn:adsk.eagle:package:38027/1"/>
 <part name="P+5" library="supply1" library_urn="urn:adsk.eagle:library:371" deviceset="+5V" device=""/>
@@
 <part name="SJ5" library="jumper" library_urn="urn:adsk.eagle:library:252" deviceset="SJ2W" device="W" package3d_urn="urn:adsk.eagle:package:15476/1"/>
 <part name="U3" library="tmc" deviceset="SSM2305" device="ADMSOP8_2" package3d_urn="urn:adsk.eagle:package:15052407/1"/>
+<part name="SJ6" library="ECE388" deviceset="SJ" device=""/>
 </parts>
 <sheets>
@@
 <net name="UCD-" class="0">
 <segment>
-<pinref part="U1" gate="G$1" pin="PE0"/>
-<wire x1="193.04" y1="106.68" x2="210.82" y2="106.68" width="0.1524" layer="91"/>
-<label x="205.74" y="106.68" size="1.778" layer="95"/>
+<pinref part="U1" gate="G$1" pin="PE1"/>
+<wire x1="193.04" y1="104.14" x2="210.82" y2="104.14" width="0.1524" layer="91"/>
+<label x="205.74" y="104.14" size="1.778" layer="95"/>
 </segment>
 </net>
 <net name="UCD+" class="0">
 <segment>
-<pinref part="U1" gate="G$1" pin="PE1"/>
-<wire x1="193.04" y1="104.14" x2="210.82" y2="104.14" width="0.1524" layer="91"/>
-<label x="205.74" y="104.14" size="1.778" layer="95"/>
+<pinref part="U1" gate="G$1" pin="PE0"/>
+<wire x1="193.04" y1="106.68" x2="210.82" y2="106.68" width="0.1524" layer="91"/>
+<label x="205.74" y="106.68" size="1.778" layer="95"/>
 </segment>
 </net>
@@
 <attribute name="VALUE" x="71.12" y="121.92" size="1.778" layer="96"/>
 </instance>
+<instance part="SJ6" gate="1" x="208.28" y="139.7" smashed="yes" rot="R90">
+<attribute name="NAME" x="205.74" y="137.16" size="1.778" layer="95" rot="R90"/>
+<attribute name="VALUE" x="212.09" y="137.16" size="1.778" layer="96" rot="R90"/>
+</instance>
 </instances>
 <busses>
@@
 <pinref part="U4" gate="G$1" pin="A"/>
 </segment>
+<segment>
+<pinref part="SJ6" gate="1" pin="2"/>
+<wire x1="208.28" y1="144.78" x2="208.28" y2="147.32" width="0.1524" layer="91"/>
+<wire x1="208.28" y1="147.32" x2="223.52" y2="147.32" width="0.1524" layer="91"/>
+<label x="208.28" y="147.32" size="1.778" layer="95"/>
+</segment>
 </net>
 <net name="N$20" class="0">
@@
 <label x="15.24" y="111.76" size="1.778" layer="95"/>
 </segment>
+<segment>
+<pinref part="SJ6" gate="1" pin="1"/>
+<wire x1="208.28" y1="134.62" x2="208.28" y2="132.08" width="0.1524" layer="91"/>
+<wire x1="208.28" y1="132.08" x2="223.52" y2="132.08" width="0.1524" layer="91"/>
+<label x="208.28" y="132.08" size="1.778" layer="95"/>
+</segment>
 </net>
 <net name="SOUND+" class="0">
@@
 <attribute name="VALUE" x="31.75" y="165.1" size="1.778" layer="96" rot="R90"/>
 </instance>
-<instance part="X17" gate="-1" x="71.12" y="157.48" smashed="yes">
-<attribute name="NAME" x="71.12" y="158.369" size="1.778" layer="95" rot="R180"/>
-</instance>
-<instance part="X17" gate="-2" x="71.12" y="152.4" smashed="yes">
-<attribute name="VALUE" x="68.58" y="148.717" size="1.778" layer="96"/>
-<attribute name="NAME" x="71.12" y="153.289" size="1.778" layer="95" rot="R180"/>
-</instance>
-<instance part="P+41" gate="1" x="78.74" y="162.56" smashed="yes">
-<attribute name="VALUE" x="81.28" y="167.64" size="1.778" layer="96" rot="R180"/>
-</instance>
-<instance part="SUPPLY73" gate="GND" x="78.74" y="147.32" smashed="yes">
-<attribute name="VALUE" x="76.835" y="144.145" size="1.778" layer="96"/>
-</instance>
 <instance part="R58" gate="G$1" x="33.02" y="106.68" smashed="yes" rot="R90">
 <attribute name="NAME" x="31.5214" y="105.41" size="1.778" layer="95" rot="R90"/>
@@
 <attribute name="VALUE" x="147.955" y="40.005" size="1.778" layer="96"/>
 </instance>
-<instance part="JP9" gate="G$1" x="182.88" y="55.88" smashed="yes">
-<attribute name="NAME" x="176.53" y="59.055" size="1.778" layer="95"/>
-<attribute name="VALUE" x="176.53" y="50.8" size="1.778" layer="96"/>
-</instance>
-<instance part="SUPPLY78" gate="GND" x="172.72" y="50.8" smashed="yes">
-<attribute name="VALUE" x="170.815" y="47.625" size="1.778" layer="96"/>
-</instance>
-<instance part="JP8" gate="G$1" x="182.88" y="68.58" smashed="yes">
-<attribute name="NAME" x="176.53" y="71.755" size="1.778" layer="95"/>
-<attribute name="VALUE" x="176.53" y="63.5" size="1.778" layer="96"/>
-</instance>
-<instance part="SUPPLY77" gate="GND" x="172.72" y="63.5" smashed="yes">
-<attribute name="VALUE" x="170.815" y="60.325" size="1.778" layer="96"/>
-</instance>
-<instance part="JP7" gate="G$1" x="182.88" y="78.74" smashed="yes">
-<attribute name="NAME" x="176.53" y="81.915" size="1.778" layer="95"/>
-<attribute name="VALUE" x="176.53" y="73.66" size="1.778" layer="96"/>
-</instance>
-<instance part="SUPPLY76" gate="GND" x="172.72" y="73.66" smashed="yes">
-<attribute name="VALUE" x="170.815" y="70.485" size="1.778" layer="96"/>
-</instance>
 <instance part="U$1" gate="G$1" x="17.78" y="154.94" smashed="yes">
 <attribute name="NAME" x="12.7" y="165.1" size="1.778" layer="95"/>
@@
 </segment>
 <segment>
-<pinref part="SUPPLY73" gate="GND" pin="GND"/>
-<pinref part="X17" gate="-2" pin="KL"/>
-<wire x1="78.74" y1="149.86" x2="78.74" y2="152.4" width="0.1524" layer="91"/>
-<wire x1="78.74" y1="152.4" x2="76.2" y2="152.4" width="0.1524" layer="91"/>
-</segment>
-<segment>
 <wire x1="27.94" y1="147.32" x2="27.94" y2="149.86" width="0.1524" layer="91"/>
 <wire x1="27.94" y1="149.86" x2="25.4" y2="149.86" width="0.1524" layer="91"/>
@@
 </segment>
 <segment>
-<pinref part="SUPPLY78" gate="GND" pin="GND"/>
-<pinref part="JP9" gate="G$1" pin="1"/>
-<wire x1="172.72" y1="53.34" x2="172.72" y2="55.88" width="0.1524" layer="91"/>
-<wire x1="172.72" y1="55.88" x2="180.34" y2="55.88" width="0.1524" layer="91"/>
-</segment>
-<segment>
-<pinref part="SUPPLY77" gate="GND" pin="GND"/>
-<pinref part="JP8" gate="G$1" pin="1"/>
-<wire x1="172.72" y1="66.04" x2="172.72" y2="68.58" width="0.1524" layer="91"/>
-<wire x1="172.72" y1="68.58" x2="180.34" y2="68.58" width="0.1524" layer="91"/>
-</segment>
-<segment>
-<pinref part="SUPPLY76" gate="GND" pin="GND"/>
-<pinref part="JP7" gate="G$1" pin="1"/>
-<wire x1="172.72" y1="76.2" x2="172.72" y2="78.74" width="0.1524" layer="91"/>
-<wire x1="172.72" y1="78.74" x2="180.34" y2="78.74" width="0.1524" layer="91"/>
-</segment>
-<segment>
 <pinref part="JP6" gate="A" pin="1"/>
 <wire x1="157.48" y1="55.88" x2="149.86" y2="55.88" width="0.1524" layer="91"/>
@@
 <wire x1="27.94" y1="172.72" x2="27.94" y2="175.26" width="0.1524" layer="91"/>
 </segment>
-<segment>
-<pinref part="X17" gate="-1" pin="KL"/>
-<pinref part="P+41" gate="1" pin="+12V"/>
-<wire x1="76.2" y1="157.48" x2="78.74" y2="157.48" width="0.1524" layer="91"/>
-<wire x1="78.74" y1="157.48" x2="78.74" y2="160.02" width="0.1524" layer="91"/>
-</segment>
 </net>

Commit message: Board Redone with notes from Ben
Parts:
- SJ4, SJ5: device jumper:SJ2WW -> jumper:SJ2W
- renumbered SW1 to RESET
Connections:
- net LED_B: now also U1.PE3; no longer U1.PB2
- net SOUND_CS: now also U1.PB2; no longer U1.PE3
- net UCD+: now also U1.PE1; no longer U1.PE0
- net UCD-: now also U1.PE0; no longer U1.PE1
Changed lines of the file:
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@@
 </variantdefs>
 <classes>
-<class number="0" name="default" width="0" drill="0">
+<class number="0" name="default" width="0.2032" drill="0.381">
+<clearance class="0" value="0.2032"/>
+</class>
+<class number="1" name="power" width="0.254" drill="0.381">
+<clearance class="1" value="0.254"/>
 </class>
 </classes>
@@
 <part name="R42" library="rcl" library_urn="urn:adsk.eagle:library:334" deviceset="R-EU_" device="R0805" package3d_urn="urn:adsk.eagle:package:23553/2" value="10K"/>
 <part name="SUPPLY38" library="supply2" library_urn="urn:adsk.eagle:library:372" deviceset="GND" device=""/>
-<part name="SW1" library="ECE388" deviceset="MOMENTARYBUTTON" device=""/>
+<part name="RESET" library="ECE388" deviceset="MOMENTARYBUTTON" device=""/>
 <part name="ISP1" library="ECE388" deviceset="AVRISP" device="-6"/>
 <part name="FRAME4" library="frames" library_urn="urn:adsk.eagle:library:229" deviceset="LETTER_L" device=""/>
@@
 <part name="H1" library="holes" library_urn="urn:adsk.eagle:library:237" deviceset="MOUNT-HOLE" device="3.0" package3d_urn="urn:adsk.eagle:package:14277/1"/>
 <part name="H2" library="holes" library_urn="urn:adsk.eagle:library:237" deviceset="MOUNT-HOLE" device="3.0" package3d_urn="urn:adsk.eagle:package:14277/1"/>
-<part name="SJ4" library="jumper" library_urn="urn:adsk.eagle:library:252" deviceset="SJ2W" device="W" package3d_urn="urn:adsk.eagle:package:15476/1"/>
-<part name="SJ5" library="jumper" library_urn="urn:adsk.eagle:library:252" deviceset="SJ2W" device="W" package3d_urn="urn:adsk.eagle:package:15476/1"/>
+<part name="SJ4" library="jumper" library_urn="urn:adsk.eagle:library:252" deviceset="SJ2W" device="" package3d_urn="urn:adsk.eagle:package:15474/1"/>
+<part name="SJ5" library="jumper" library_urn="urn:adsk.eagle:library:252" deviceset="SJ2W" device="" package3d_urn="urn:adsk.eagle:package:15474/1"/>
 <part name="U3" library="tmc" deviceset="SSM2305" device="ADMSOP8_2" package3d_urn="urn:adsk.eagle:package:15052407/1"/>
 <part name="SJ6" library="ECE388" deviceset="SJ" device=""/>
@@
 <attribute name="VALUE" x="110.744" y="140.081" size="1.778" layer="96"/>
 </instance>
-<instance part="SW1" gate="G$1" x="96.52" y="119.38" smashed="yes"/>
+<instance part="RESET" gate="G$1" x="96.52" y="119.38" smashed="yes"/>
 <instance part="ISP1" gate="G$1" x="33.02" y="35.56" smashed="yes">
 <attribute name="NAME" x="38.1" y="40.64" size="1.778" layer="95"/>
@@
 </segment>
 <segment>
-<pinref part="SW1" gate="G$1" pin="A1"/>
+<pinref part="RESET" gate="G$1" pin="A1"/>
 <pinref part="SUPPLY4" gate="GND" pin="GND"/>
 <wire x1="99.06" y1="124.46" x2="93.98" y2="124.46" width="0.1524" layer="91"/>
@@
 </segment>
 <segment>
-<wire x1="193.04" y1="142.24" x2="210.82" y2="142.24" width="0.1524" layer="91"/>
-<label x="203.2" y="142.24" size="1.778" layer="95"/>
-<pinref part="U1" gate="G$1" pin="PB2"/>
-</segment>
-<segment>
 <pinref part="R2" gate="G$1" pin="1"/>
 <wire x1="88.9" y1="165.1" x2="88.9" y2="160.02" width="0.1524" layer="91"/>
@@
 <label x="71.12" y="160.02" size="1.778" layer="95"/>
 </segment>
+<segment>
+<wire x1="193.04" y1="99.06" x2="210.82" y2="99.06" width="0.1524" layer="91"/>
+<pinref part="U1" gate="G$1" pin="PE3"/>
+<label x="203.2" y="99.06" size="1.778" layer="95"/>
+</segment>
 </net>
 <net name="LED_O" class="0">
@@
 </segment>
 <segment>
-<wire x1="193.04" y1="99.06" x2="210.82" y2="99.06" width="0.1524" layer="91"/>
-<pinref part="U1" gate="G$1" pin="PE3"/>
-<label x="198.12" y="99.06" size="1.778" layer="95"/>
+<wire x1="193.04" y1="142.24" x2="210.82" y2="142.24" width="0.1524" layer="91"/>
+<label x="198.12" y="142.24" size="1.778" layer="95"/>
+<pinref part="U1" gate="G$1" pin="PB2"/>
 </segment>
 </net>
@@
 <wire x1="132.08" y1="137.16" x2="116.84" y2="137.16" width="0.1524" layer="91"/>
 <pinref part="C1" gate="G$1" pin="1"/>
-<pinref part="SW1" gate="G$1" pin="B1"/>
+<pinref part="RESET" gate="G$1" pin="B1"/>
 <wire x1="119.38" y1="124.46" x2="137.16" y2="124.46" width="0.1524" layer="91"/>
 <wire x1="137.16" y1="124.46" x2="137.16" y2="137.16" width="0.1524" layer="91"/>
@@
 <net name="UCD-" class="0">
 <segment>
-<pinref part="U1" gate="G$1" pin="PE1"/>
-<wire x1="193.04" y1="104.14" x2="210.82" y2="104.14" width="0.1524" layer="91"/>
-<label x="205.74" y="104.14" size="1.778" layer="95"/>
+<pinref part="U1" gate="G$1" pin="PE0"/>
+<wire x1="193.04" y1="106.68" x2="210.82" y2="106.68" width="0.1524" layer="91"/>
+<label x="205.74" y="106.68" size="1.778" layer="95"/>
 </segment>
 </net>
 <net name="UCD+" class="0">
 <segment>
-<pinref part="U1" gate="G$1" pin="PE0"/>
-<wire x1="193.04" y1="106.68" x2="210.82" y2="106.68" width="0.1524" layer="91"/>
-<label x="205.74" y="106.68" size="1.778" layer="95"/>
+<pinref part="U1" gate="G$1" pin="PE1"/>
+<wire x1="193.04" y1="104.14" x2="210.82" y2="104.14" width="0.1524" layer="91"/>
+<label x="205.74" y="104.14" size="1.778" layer="95"/>
 </segment>
 </net>
@@
 </segment>
 </net>
-<net name="+12V" class="0">
+<net name="+12V" class="1">
 <segment>
 <pinref part="R13" gate="G$1" pin="2"/>
@@
 </segment>
 </net>
-<net name="+12V" class="0">
+<net name="+12V" class="1">
 <segment>
 <pinref part="SJ2" gate="G$1" pin="3"/>
@@
 </segment>
 </net>
-<net name="N$19" class="0">
+<net name="N$19" class="1">
 <segment>
 <pinref part="JP5" gate="A" pin="1"/>
